Commit message: Bug fixes: turtlebot and sl_ur_demo

File: ros_humble/Ubuntu/src/sl_ur_demo/ur_description/meshes/stand/urdf/stand.urdf (robot description, URDF)
Before this commit: robot stand, 2 links, 1 joints
Links:
- link stand_link: geometry collision mesh filename=model://stand/meshes/binPickingStand_scaled.dae; visual mesh filename=model://stand/meshes/binPickingStand_scaled.dae
